File: 001 PCB/KICAD/TheENDGAME2024.kicad_sch (KiCad schematic)
At the start: 74 parts, among them SW10 SW_Push, SW11 SW_Push, SW12 SW_Push, SW13 SW_Push, SW14 SW_Push, SW15 SW_Push, SW16 SW_Push, SW17 SW_Push, SW18 SW_Push, SW19 SW_Push, SW2 SW_Push, SW20 SW_Push, SW21 SW_Push, SW22 SW_Push, SW23 SW_Push, SW24 SW_Push, SW25 SW_Push, SW26 SW_Push, SW27 SW_Push, SW28 SW_Push, SW29 SW_Push, SW3 SW_Push, SW30 SW_Push, SW31 SW_Push, SW32 SW_Push, SW33 SW_Push, SW34 SW_Push, SW35 SW_Push, SW36 SW_Push, SW37 SW_Push, SW4 SW_Push, SW5 SW_Push, SW6 SW_Push, SW7 SW_Push, SW8 SW_Push, SW9 SW_Push, U2 RP2040-Zero_stolen_from_Purox

Commit message: upload new pics
Parts:
- BZ2: symbol Best Symbol Library Final v3:Buzzer -> TheEndgame2024:Buzzer
- D10, D11, D12, D13, D14, D15, D17, D18, D19, D20, D22, D23, D24, D25, D26, D27, D28, D29, D32, D33, D34, D35, D36, D37, D38, D39, D40, D41, D44, D45, D46, D47, D5, D6, D7, D8: symbol ENDGAME_UWU_Gatekeeper_stuff:D_Small -> TheEndgame2024:D_Small
- SW10, SW11, SW12, SW13, SW14, SW15, SW16, SW17, SW18, SW19, SW2, SW20, SW21, SW22, SW23, SW24, SW25, SW26, SW27, SW28, SW29, SW3, SW30, SW31, SW32, SW33, SW34, SW35, SW36, SW37, SW4, SW5, SW6, SW7, SW8, SW9: symbol ENDGAME_UWU_Gatekeeper_stuff:SW_Push -> TheEndgame2024:SW_Push
- U2: symbol Best Symbol Library Final v3:RP2040-Zero_stolen_from_Purox -> TheEndgame2024:RP2040-Zero_stolen_from_Purox
